File: pcb/morseboard-8088/output.kicad_sch (KiCad schematic)
At the start: 56 parts, among them J2 CLKSRC, SW2 MANCLK, U10 74HC273, U11 74HC123, U6 74HC138

Commit message: Adding source and revising PCB
Connections:
- net AD16 renamed A16
- net AD17 renamed A17
- net AD18 renamed A18
- net AD19 renamed A19

Commit message: Revising testboard
Parts:
- removed C17: 100uF, Capacitor_THT:CP_Radial_D6.3mm_P2.50mm, symbol Device:C_Polarized
- removed C18: 100nF, Capacitor_THT:C_Disc_D5.0mm_W2.5mm_P5.00mm, symbol Device:C
- removed C19: 1uF, Capacitor_THT:CP_Radial_D5.0mm_P2.50mm, symbol Device:C_Polarized
- removed D1, D10, D11, D12, D13, D14, D15, D16, D17, D18, D19, D2, D20, D21, D22, D23, D24, D25, D26, D27, D28, D29, D3, D30, D31, D32, D33, D34, D35, D36, D37, D38, D39, D4, D40, D41, D5, D6, D7, D8: LED, LED_THT:LED_D5.0mm, symbol Device:LED
- removed J2: CLKSRC, Connector_PinHeader_2.54mm:PinHeader_1x03_P2.54mm_Vertical, symbol Connector:Conn_01x03_Pin
- removed R3, R5: 10k, Resistor_THT:R_Axial_DIN0207_L6.3mm_D2.5mm_P7.62mm_Horizontal, symbol Device:R
- removed R4: 47k, Resistor_THT:R_Axial_DIN0207_L6.3mm_D2.5mm_P7.62mm_Horizontal, symbol Device:R
- removed RN1, RN2, RN3, RN4, RN5: 510, Resistor_THT:R_Array_SIP9, symbol Device:R_Network08_Split
- removed SW2: MANCLK, Button_Switch_THT:SW_PUSH_6mm, symbol Switch:SW_Push
- removed U11: 74HC123, Package_DIP:DIP-16_W7.62mm_Socket, symbol 74xx:74HC123
- U10: value 74HC273 -> 74HCT273
- U6: value 74HC138 -> 74HCT138
Connections:
- no-connect marks 9 -> 7
Other:
- note removed: "10k resistor with 1uF cap gives 0.45*RC = 0.45*0.01s = 0.0045s active low pulse"
- note removed: "47k resistor with 100uF cap gives t = 0.45RC = 0.45*4.7s= 2.115s delay between consecutive button presses"
- note removed: "Soft reset"
