File: pcb/morseboard-8088/_autosave-morseboard-8088.kicad_sch (KiCad schematic)
At the start: 64 parts, among them J1 USB_B, J2 UART1, J3 TxD, J4 ~{CTS}, J5 RxD, J6 ~{RTS}, SW1 SW_SPDT, SW2 INTPORT, SW4 NMI, SW6 RESET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

Commit message: Fixing bugs in PCB design
Parts:
- removed J3: TxD, Connector_PinHeader_2.54mm:PinHeader_1x03_P2.54mm_Vertical, symbol Connector:Conn_01x03_Pin
- removed J4: ~{CTS}, Connector_PinHeader_2.54mm:PinHeader_1x03_P2.54mm_Vertical, symbol Connector:Conn_01x03_Pin
- removed J5: RxD, Connector_PinHeader_2.54mm:PinHeader_1x03_P2.54mm_Vertical, symbol Connector:Conn_01x03_Pin
- removed J6: ~{RTS}, Connector_PinHeader_2.54mm:PinHeader_1x03_P2.54mm_Vertical, symbol Connector:Conn_01x03_Pin
Connections:
- net R1IN is gone; now on net UART3: U13.13 (R1IN)
- net R2IN is gone; now on net UART7: U13.8 (R2IN)
- net T1OUT is gone; now on net UART2: U13.14 (T1OUT)
- net T2OUT is gone; now on net UART8: U13.7 (T2OUT)
