File: pcb/mb88-testboard/mb88-testboard.kicad_sch (KiCad schematic)
At the start: 33 parts, among them J1 USB_B, SW1 SW_SPDT, SW3 RES, SW4 NMI, U1 8088, U2 74HCT573, U3 74HCT573, U4 74HCT245, U5 SST39SF040, U7 74HCT02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

Commit message: Revising testboard
Other:
- title: (none) -> Morse Board 8088 TEST BOARD
Changed lines of the file:
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@@
 	(generator_version "9.0")
 	(paper "A4")
+	(title_block
+		(title "Morse Board 8088 TEST BOARD")
+		(date "2025-05-21")
+		(rev "1")
+	)
 	(text "Board-wide power-switch\n"
 		(exclude_from_sim no)
@@
 		)
 		(instances
-			(project "morseboard-8088"
+			(project "mb88-testboard"
 				(path "/27cb38f9-12de-466e-a080-2dfa091752ed"
 					(page "2")

Commit message: Initial commit TL16C550
Parts:
- U1: footprint Package_DIP:DIP-40_W15.24mm -> Package_DIP:DIP-40_W15.24mm_Socket
- U9: footprint Package_DIP:DIP-32_W15.24mm -> Package_DIP:DIP-32_W15.24mm_Socket
Changed lines of the file:
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@@
 			)
 		)
-		(property "Footprint" "Package_DIP:DIP-32_W15.24mm"
+		(property "Footprint" "Package_DIP:DIP-32_W15.24mm_Socket"
 			(at 189.23 52.07 0)
 			(effects
@@
 			)
 		)
-		(property "Footprint" "Package_DIP:DIP-40_W15.24mm"
+		(property "Footprint" "Package_DIP:DIP-40_W15.24mm_Socket"
 			(at 44.45 67.31 0)
 			(effects
