File: pcb/morseboard-8088-vera/controller.kicad_sch (KiCad schematic)
At the start: 19 parts, among them J4 Mini-DIN-6, J5 Conn_01x03_Pin, SW5 ON, SW6 RESET, U12 ATmega328P-P, U14 74HCT245, U7 74HCT02, Y1 Crystal

Commit message: The quest continues
Parts:
- removed U7: 74HCT02, Package_DIP:DIP-14_W7.62mm_Socket, symbol 74xx:74HC02
Connections:
- net ~{CTRL_CE}: now reaches U14.19 (CE)
- net INTR: no longer names the net of U12.15 (PB1)
- net SERIAL_INT: no longer names the net of U12.5 (PD3)
- net VERA_INT: no longer names the net of U12.17 (PB3)
- net ~{INTA}: no longer names the net of U12.16 (PB2)
- net ~{IO03}: no longer names the net of U12.18 (PB4)
- no-connect marks 2 -> 7
Other:
- note removed: "KB"
