File: pcb/morseboard-8088-vera/morseboard-8088-vera.kicad_sch (KiCad schematic)
At the start: 55 parts, among them J1 USB_B, J2 UART1, J3 Bus, SW1 SW_SPDT, SW4 NMI, U1 8088, U10 74HCT273, U11 TL16C550, U13 MAX232, U2 74HCT573, U3 74HCT573, U4 74HCT245, U5 SST39SF040, U6 74HCT138, U7 74HCT02, U8 74HCT00, U9 AS6C4008-55PCN, X1 7.3728 MHz

Commit message: The quest continues
Parts:
- removed U6: 74HCT138, Package_DIP:DIP-16_W7.62mm_Socket, symbol 74xx:74HC138
- removed U7: 74HCT02, Package_DIP:DIP-14_W7.62mm_Socket, symbol 74xx:74HC02
- removed U8: 74HCT00, Package_DIP:DIP-14_W7.62mm_Socket, symbol 74xx:74HC00
- added C33, C34, C35, C36: 100nF, Capacitor_THT:C_Disc_D5.0mm_W2.5mm_P5.00mm, symbol Device:C
- added J6: Atmel-JTAG-10, Connector_IDC:IDC-Header_2x05_P2.54mm_Vertical, symbol atf1504_plcc44_breakout:Atmel-JTAG-10
- added U23: ATF1504AS, Package_LCC:PLCC-44_THT-Socket, symbol atf1504_plcc44_breakout:ATF1504AS-xJx44
Connections:
- net A19: now also U23.14 (I/O)
- net A5: now also U23.6 (I/O)
- net A6: now also U23.8 (I/O)
- net A7: now also U23.9 (I/O)
- net D0: now also U23.18 (I/O)
- net D1: now also U23.19 (I/O)
- net D2: now also U23.20 (I/O)
- net D3: now also U23.21 (I/O)
- net D4: now also U23.24 (I/O)
- net D5: now also U23.25 (I/O/PD2)
- net D6: now also U23.26 (I/O)
- net D7: now also U23.27 (I/O)
- net GND: now also C33.2, C34.2, C35.2, C36.2, J6.10 (GND), J6.2 (GND), U23.10 (GND), U23.22 (GND), U23.30 (GND), U23.42 (GND)
- net INTR: now also U23.36 (I/O)
- net LATCH: now also U23.37 (I/O)
- net RES: now also U23.31 (I/O)
- net SERIAL_INT: now also U23.33 (I/O)
- net VCC: now also C33.1, C34.1, C35.1, C36.1, J6.4 (VccT), U23.15 (VCC), U23.23 (VCC), U23.3 (VCC), U23.35 (VCC)
- net VERA_INT: now also U23.34 (I/O)
- net ~{INTA}: now also U23.5 (I/O)
- net ~{IO}/M: now also U23.4 (I/O)
- net ~{RAMCS}: now also U23.40 (I/O)
- net ~{RD}: now also U23.11 (I/O/PD1)
- net ~{RES}: now also U23.1 (I/GCLR)
- net ~{ROMCS}: now also U23.41 (I/O/GCLK3)
- net ~{WR}: now also U23.12 (I/O)
- net ~{IO01} renamed ~{SERIAL_CE}
- net ~{SERIAL_CE}: now also U23.29 (I/O)
- new net TCK: J6.1 (TCK), U23.32 (I/O/TCK)
- new net TDI: J6.9 (TDI), U23.7 (I/O/TDI)
- new net TDO: J6.3 (TDO), U23.38 (I/O/TDO)
- new net TMS: J6.5 (TMS), U23.13 (I/O/TMS)
- new net ~{CTRL_CE}: U23.39 (I/O)
- no-connect marks 30 -> 32
Other:
- note removed: "0x00: LED"
- note removed: "0x20: SERIAL"
- note removed: "0x40: VERA"
- note removed: "0x60: KB"
- note removed: "Do not output on ~{INTA}!"
